File: KiCad/THW_bagde.kicad_sch (KiCad schematic)
At the start: 41 parts, among them J1 USB_B, J2 ISP, SW1 SW_Push, SW2 SW_Push, SW3 SW_Push, U1 ATmega328-P, Y1 Crystal

Commit message: switching to plain avr lib instead arduino framework
Parts:
- added C?: 100n, Capacitor_THT:C_Disc_D3.8mm_W2.6mm_P2.50mm, symbol Device:C
- C3: value C -> 100n
Connections:
- net +5V: now also C?.1
- net GND: now also C?.2
Changed lines of the file:
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@@
   (junction (at 207.01 81.915) (diameter 0) (color 0 0 0 0)
   )
+  (junction (at 49.53 45.72) (diameter 0) (color 0 0 0 0)
+  )
   (junction (at 181.61 81.915) (diameter 0) (color 0 0 0 0)
   )
-  (junction (at 49.53 45.847) (diameter 0) (color 0 0 0 0)
-  )
   (junction (at 240.665 129.667) (diameter 0) (color 0 0 0 0)
   )
@@
   (junction (at 81.28 112.395) (diameter 0) (color 0 0 0 0)
   )
+  (junction (at 41.275 45.72) (diameter 0) (color 0 0 0 0)
+  )
   (junction (at 81.28 99.06) (diameter 0) (color 0 0 0 0)
   )
@@
   )
   (junction (at 155.194 143.764) (diameter 0) (color 0 0 0 0)
+  )
+  (junction (at 37.465 59.055) (diameter 0) (color 0 0 0 0)
   )
   (junction (at 121.285 102.87) (diameter 0) (color 0 0 0 0)
@@
     (stroke (width 0) (type default) (color 0 0 0 0))
   )
+  (wire (pts (xy 34.29 59.055) (xy 37.465 59.055))
+    (stroke (width 0) (type default) (color 0 0 0 0))
+  )
   (wire (pts (xy 262.636 140.462) (xy 262.636 143.764))
     (stroke (width 0) (type default) (color 0 0 0 0))
@@
     (stroke (width 0) (type default) (color 0 0 0 0))
   )
-  (wire (pts (xy 41.275 56.642) (xy 41.275 58.547))
+  (wire (pts (xy 41.275 56.642) (xy 41.275 59.055))
     (stroke (width 0) (type default) (color 0 0 0 0))
   )
@@
     (stroke (width 0) (type default) (color 0 0 0 0))
   )
-  (wire (pts (xy 52.07 45.847) (xy 52.07 66.675))
+  (wire (pts (xy 52.07 45.72) (xy 52.07 66.675))
     (stroke (width 0) (type default) (color 0 0 0 0))
   )
@@
     (stroke (width 0) (type default) (color 0 0 0 0))
   )
-  (wire (pts (xy 49.53 42.672) (xy 49.53 45.847))
+  (wire (pts (xy 49.53 42.672) (xy 49.53 45.72))
     (stroke (width 0) (type default) (color 0 0 0 0))
   )
@@
     (stroke (width 0) (type default) (color 0 0 0 0))
   )
+  (wire (pts (xy 34.29 45.72) (xy 41.275 45.72))
+    (stroke (width 0) (type default) (color 0 0 0 0))
+  )
   (wire (pts (xy 93.218 66.675) (xy 95.25 66.675))
     (stroke (width 0) (type default) (color 0 0 0 0))
   )
-  (wire (pts (xy 52.07 45.847) (xy 49.53 45.847))
+  (wire (pts (xy 52.07 45.72) (xy 49.53 45.72))
     (stroke (width 0) (type default) (color 0 0 0 0))
   )
@@
     (stroke (width 0) (type default) (color 0 0 0 0))
   )
+  (wire (pts (xy 34.29 56.515) (xy 34.29 59.055))
+    (stroke (width 0) (type default) (color 0 0 0 0))
+  )
   (wire (pts (xy 116.84 56.515) (xy 116.84 61.595))
     (stroke (width 0) (type default) (color 0 0 0 0))
@@
     (stroke (width 0) (type default) (color 0 0 0 0))
   )
-  (wire (pts (xy 41.275 45.847) (xy 41.275 49.022))
+  (wire (pts (xy 41.275 45.72) (xy 41.275 49.022))
     (stroke (width 0) (type default) (color 0 0 0 0))
   )
@@
     (stroke (width 0) (type default) (color 0 0 0 0))
   )
-  (wire (pts (xy 49.53 45.847) (xy 49.53 66.675))
+  (wire (pts (xy 49.53 45.72) (xy 49.53 66.675))
     (stroke (width 0) (type default) (color 0 0 0 0))
   )
@@
     (stroke (width 0) (type default) (color 0 0 0 0))
   )
+  (wire (pts (xy 37.465 59.055) (xy 41.275 59.055))
+    (stroke (width 0) (type default) (color 0 0 0 0))
+  )
   (wire (pts (xy 207.01 81.915) (xy 212.09 81.915))
     (stroke (width 0) (type default) (color 0 0 0 0))
@@
     (stroke (width 0) (type default) (color 0 0 0 0))
   )
+  (wire (pts (xy 34.29 48.895) (xy 34.29 45.72))
+    (stroke (width 0) (type default) (color 0 0 0 0))
+  )
   (wire (pts (xy 171.45 81.915) (xy 181.61 81.915))
     (stroke (width 0) (type default) (color 0 0 0 0))
@@
     (stroke (width 0) (type default) (color 0 0 0 0))
   )
-  (wire (pts (xy 49.53 45.847) (xy 41.275 45.847))
+  (wire (pts (xy 49.53 45.72) (xy 41.275 45.72))
     (stroke (width 0) (type default) (color 0 0 0 0))
   )
@@
   )
   (wire (pts (xy 64.77 102.235) (xy 74.93 102.235))
+    (stroke (width 0) (type default) (color 0 0 0 0))
+  )
+  (wire (pts (xy 37.465 59.055) (xy 37.465 60.325))
     (stroke (width 0) (type default) (color 0 0 0 0))
   )
@@
     )
     (property "Datasheet" "~" (id 3) (at 232.41 50.8 0)
+      (effects (font (size 1.27 1.27)) hide)
+    )
+    (pin "1")
+    (pin "2")
+  )
+  (symbol (lib_id "Device:C") (at 34.29 52.705 0) (unit 1)
+    (in_bom yes) (on_board yes)
+    (property "Reference" "C?" (id 0) (at 36.83 51.435 0)
+      (effects (font (size 1.27 1.27)) (justify left))
+    )
+    (property "Value" "100n" (id 1) (at 36.83 53.975 0)
+      (effects (font (size 1.27 1.27)) (justify left))
+    )
+    (property "Footprint" "Capacitor_THT:C_Disc_D3.8mm_W2.6mm_P2.50mm" (id 2) (at 35.2552 56.515 0)
+      (effects (font (size 1.27 1.27)) hide)
+    )
+    (property "Datasheet" "~" (id 3) (at 34.29 52.705 0)
       (effects (font (size 1.27 1.27)) hide)
     )
@@
     (pin "2")
   )
-  (symbol (lib_id "power:GND") (at 41.275 58.547 0) (unit 1)
-    (in_bom yes) (on_board yes)
-    (property "Reference" "#PWR0103" (id 0) (at 41.275 64.897 0)
-      (effects (font (size 1.27 1.27)) hide)
-    )
-    (property "Value" "GND" (id 1) (at 41.275 62.357 0))
-    (property "Footprint" "" (id 2) (at 41.275 58.547 0)
-      (effects (font (size 1.27 1.27)) hide)
-    )
-    (property "Datasheet" "" (id 3) (at 41.275 58.547 0)
+  (symbol (lib_id "power:GND") (at 37.465 60.325 0) (unit 1)
+    (in_bom yes) (on_board yes)
+    (property "Reference" "#PWR0103" (id 0) (at 37.465 66.675 0)
+      (effects (font (size 1.27 1.27)) hide)
+    )
+    (property "Value" "GND" (id 1) (at 37.465 64.135 0))
+    (property "Footprint" "" (id 2) (at 37.465 60.325 0)
+      (effects (font (size 1.27 1.27)) hide)
+    )
+    (property "Datasheet" "" (id 3) (at 37.465 60.325 0)
       (effects (font (size 1.27 1.27)) hide)
     )
@@
       (effects (font (size 1.27 1.27)) (justify left))
     )
-    (property "Value" "C" (id 1) (at 43.815 54.102 0)
+    (property "Value" "100n" (id 1) (at 43.815 54.102 0)
       (effects (font (size 1.27 1.27)) (justify left))
     )
@@
     )
     (path "/fd3196b5-c704-4abc-acec-f5b4e906b39f"
-      (reference "C3") (unit 1) (value "C") (footprint "Capacitor_THT:C_Disc_D3.8mm_W2.6mm_P2.50mm")
+      (reference "C3") (unit 1) (value "100n") (footprint "Capacitor_THT:C_Disc_D3.8mm_W2.6mm_P2.50mm")
     )
     (path "/49c94512-f34b-41f9-b444-517e32ec6cd9"
@@
       (reference "C7") (unit 1) (value "C") (footprint "Capacitor_THT:C_Disc_D3.8mm_W2.6mm_P2.50mm")
     )
+    (path "/2f2829fb-8b12-4181-a98c-c947e241ad97"
+      (reference "C?") (unit 1) (value "100n") (footprint "Capacitor_THT:C_Disc_D3.8mm_W2.6mm_P2.50mm")
+    )
     (path "/a7385d01-bac2-4df6-adcf-5e26bcc0c5b7"

Commit message: first tests with tks-badge firmware
Parts:
- gave numbers to parts that had none: 1
Connections:
- net PC1: now also R7.1; no longer R6.1
- net PC2: now also R8.1; no longer R7.1
- net PC3: now also R9.1; no longer R8.1
- net PC4: now also R10.1; no longer R9.1
- net PC0: now reaches U1.23 (PC0)
- net PC0: now also R6.1
- net PC5: no longer names the net of U1.28 (PC5)
- net PC5: no longer R10.1
- no-connect marks 3 -> 4
Changed lines of the file:
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@@
   (junction (at 121.285 96.52) (diameter 0) (color 0 0 0 0)
   )
+  (no_connect (at 64.77 109.855))
   (no_connect (at 34.29 74.295))
   (no_connect (at 164.084 134.239))
@@
     (stroke (width 0) (type default) (color 0 0 0 0))
   )
+  (wire (pts (xy 64.77 97.155) (xy 74.93 97.155))
+    (stroke (width 0) (type default) (color 0 0 0 0))
+  )
   (wire (pts (xy 64.77 122.555) (xy 74.803 122.555))
     (stroke (width 0) (type default) (color 0 0 0 0))
@@
     (stroke (width 0) (type default) (color 0 0 0 0))
   )
-  (wire (pts (xy 64.77 109.855) (xy 74.93 109.855))
-    (stroke (width 0) (type default) (color 0 0 0 0))
-  )
   (polyline (pts (xy 137.16 28.575) (xy 25.4 28.575))
     (stroke (width 0) (type default) (color 0 0 0 0))
@@
     (effects (font (size 1.27 1.27)) (justify right bottom))
   )
-  (label "PC5" (at 252.73 38.1 180)
+  (label "PC4" (at 252.73 38.1 180)
     (effects (font (size 1.27 1.27)) (justify right bottom))
   )
@@
     (effects (font (size 1.27 1.27)) (justify right bottom))
   )
-  (label "PC5" (at 74.93 109.855 180)
+  (label "PC0" (at 74.93 97.155 180)
     (effects (font (size 1.27 1.27)) (justify right bottom))
   )
@@
     (effects (font (size 1.27 1.27)) (justify right bottom))
   )
-  (label "PC1" (at 212.09 38.1 180)
+  (label "PC0" (at 212.09 38.1 180)
     (effects (font (size 1.27 1.27)) (justify right bottom))
   )
@@
     (effects (font (size 1.27 1.27)) (justify left bottom))
   )
-  (label "PC3" (at 232.41 38.1 180)
+  (label "PC2" (at 232.41 38.1 180)
     (effects (font (size 1.27 1.27)) (justify right bottom))
   )
@@
     (effects (font (size 1.27 1.27)) (justify left bottom))
   )
-  (label "PC4" (at 242.57 38.1 180)
+  (label "PC3" (at 242.57 38.1 180)
     (effects (font (size 1.27 1.27)) (justify right bottom))
   )
@@
     (effects (font (size 1.27 1.27)) (justify right bottom))
   )
-  (label "PC2" (at 222.25 38.1 180)
+  (label "PC1" (at 222.25 38.1 180)
     (effects (font (size 1.27 1.27)) (justify right bottom))
   )
@@
   (symbol (lib_id "Device:C") (at 34.29 52.705 0) (unit 1)
     (in_bom yes) (on_board yes)
-    (property "Reference" "C?" (id 0) (at 36.83 51.435 0)
+    (property "Reference" "C8" (id 0) (at 36.83 51.435 0)
       (effects (font (size 1.27 1.27)) (justify left))
     )
@@
     )
     (path "/2f2829fb-8b12-4181-a98c-c947e241ad97"
-      (reference "C?") (unit 1) (value "100n") (footprint "Capacitor_THT:C_Disc_D3.8mm_W2.6mm_P2.50mm")
+      (reference "C8") (unit 1) (value "100n") (footprint "Capacitor_THT:C_Disc_D3.8mm_W2.6mm_P2.50mm")
     )
     (path "/a7385d01-bac2-4df6-adcf-5e26bcc0c5b7"
