File: KiCad/THW_bagde.kicad_pcb (KiCad board)
At the start: 2 copper layers, 84.9 x 82.9 mm, 52 parts, among them J1 USB_B, J2 ICSP, SW1 SW_Push, SW2 SW_Push, SW3 SW_Push, U1 ATmega328-P, Y1 Crystal

Commit message: Adding Rendering of bottom and adding QR to GitHub Repo.
Parts:
- added G***: LOGO, LOGO, B.Cu at (151.7, 124.9)

Commit message: first order
Parts:
- removed the G*** at (151.7, 124.9)
Routing:
- net Net-(D6-Pad2): track 51.8 -> 53.3 mm
- net Net-(D5-Pad2): track 52.9 -> 53.8 mm
